Commit message: initial proof of concept vel ctrl

File: common/test/urdf/acrobat_robot.urdf (robot description, URDF)
Before this commit: robot acrobat, 3 links, 2 joints
Joints:
- joint joint1: limit (none) -> lower=-3.14159265359 upper=3.14159265359 effort=50.0 velocity=1.0; type continuous -> revolute

File: common/test/urdf/acrobat_robot.urdf.xacro (robot description, xacro)
@@ -8,4 +8,5 @@
   <xacro:property name="height2" value="1" /> <!-- Link 2 -->
   <xacro:property name="axel_offset" value="0.05" /> <!-- Space btw top of beam and the each joint -->
+  <xacro:property name="M_PI" value="3.141592653589793" />
   <!-- Tags needed for rviz to color model -->
   <xacro:include filename="$(find pybullet_ros)/common/test/urdf/materials.urdf.xacro" />
@@ -40,10 +41,10 @@
     </inertial>
   </link>
-  <joint name="joint1" type="continuous">
+  <joint name="joint1" type="revolute">
     <parent link="link1"/>
     <child link="link2"/>
+    <limit effort="50.0" lower="${-M_PI}" upper="${M_PI}" velocity="1.0"/>
+    <axis xyz="0 1 0"/>
     <origin xyz="0 ${width} ${height1 - axel_offset}" rpy="0 0 0"/>
-    <axis xyz="0 1 0"/>
-    <dynamics damping="0.7"/>
   </joint>
   <!-- Acrobat green link -->

Commit message: done with velocity control

File: common/test/urdf/acrobat_robot.urdf (robot description, URDF)
Before this commit: robot acrobat, 3 links, 2 joints
Joints:
- joint joint1: limit lower=-3.14159265359 upper=3.14159265359 effort=50.0 velocity=1.0 -> lower=-3.14159265359 upper=3.14159265359 effort=1500.0 velocity=100.0

File: common/test/urdf/acrobat_robot.urdf.xacro (robot description, xacro)
@@ -44,5 +44,5 @@
     <parent link="link1"/>
     <child link="link2"/>
-    <limit effort="50.0" lower="${-M_PI}" upper="${M_PI}" velocity="1.0"/>
+    <limit effort="1500.0" lower="${-M_PI}" upper="${M_PI}" velocity="100.0"/>
     <axis xyz="0 1 0"/>
     <origin xyz="0 ${width} ${height1 - axel_offset}" rpy="0 0 0"/>
