Commit message: code refactor, add r2d2 launch file and urdf model

File: common/test/urdf/r2d2/r2d2.urdf (robot description, URDF)
Before this commit: robot r2d2, 18 links, 17 joints
Links:
- removed link base_footprint
- removed link laser_link
Joints:
- removed joint base_link_to_laser_joint
- removed joint footprint_to_base_link

Commit message: add 90 degree rotation of r2r2 to face forward when commanded to go forward

File: common/test/urdf/r2d2/r2d2.urdf (robot description, URDF)
Before this commit: robot physics, 16 links, 15 joints
Links:
- added link base_footprint
Joints:
- added joint footprint_to_base_link: type fixed, parent base_footprint, child base_link, origin xyz=0 0 0 rpy=0 0 -1.57075
