Commit message: adjust mass and tip link of example robot, add generated urdf

File: common/test/urdf/acrobat_robot/acrobat_robot.urdf (robot description, URDF)
Before this commit: robot acrobat, 3 links, 2 joints
Links:
- removed link world
- added link base_link, mass 0.1; collision cylinder length=0.15 radius=0.15; visual cylinder length=0.15 radius=0.15
- added link link1_tip
- added link odom
- added link static_link1
- added link tip_link
- link link1: mass 1 -> 0.1; geometry collision box size=0.1 0.1 1.0; visual box size=0.1 0.1 1.6
- link link2: mass 1 -> 0.1; geometry collision box size=0.1 0.1 1.2; visual box size=0.1 0.1 1.2
Joints:
- removed joint fixed
- removed joint joint1
- added joint base_link_to_static_link1: type fixed, parent base_link, child static_link1, origin xyz=0 0 0.15 rpy=0 0 0
- added joint link1_tip_to_link2: type revolute, parent link1_tip, child link2, origin xyz=0 0 0 rpy=0 0 0, axis 0 1 0, limit lower=-3.14159265359 upper=3.14159265359 effort=1500.0 velocity=100.0
- added joint link1_to_link1_tip: type fixed, parent link1, child link1_tip, origin xyz=0 0 1.6 rpy=0 0 0
- added joint link1_to_static_link1: type revolute, parent static_link1, child link1, origin xyz=0 0 0 rpy=0 0 0, axis 0 1 0, limit lower=-3.14159265359 upper=3.14159265359 effort=1500.0 velocity=100.0
- added joint link2_to_tip_link: type fixed, parent link2, child tip_link, origin xyz=0 0 1.15 rpy=0 0 0
- added joint odom_to_base_link: type revolute, parent odom, child base_link, origin xyz=0 0 0 rpy=0 0 0, axis 0 0 1, limit lower=-3.14159265359 upper=3.14159265359 effort=1500.0 velocity=100.0

File: common/test/urdf/acrobat_robot/acrobat_robot.urdf.xacro (robot description, xacro)
@@ -3,5 +3,5 @@
 <robot name="acrobat" xmlns:xacro="http://www.ros.org/wiki/xacro">
   <!-- Constants for robot dimensions -->
-  <xacro:property name="mass" value="1" /> <!-- arbitrary value for mass -->
+  <xacro:property name="mass" value="0.1" /> <!-- arbitrary value for mass -->
   <xacro:property name="width" value="0.1" /> <!-- Square dimensions (widthxwidth) of beams -->
   <xacro:property name="height1" value="1.6" /> <!-- Link 1: 0.1768 -->
@@ -56,5 +56,5 @@
       <origin xyz="0 0 ${height1/2}" rpy="0 0 0"/>
       <geometry>
-        <box size="${width} ${width} ${height1}"/>
+        <box size="${width} ${width} ${height1-0.6}"/>
       </geometry>
     </collision>
