Commit message: add laser scanner to r2d2, remove gripper

File: common/test/urdf/r2d2_robot/r2d2.urdf.xacro (robot description, xacro)
@@ -1,4 +1,10 @@
 <?xml version="1.0"?>
-<robot name="r2d2">
+<robot name="r2d2" xmlns:xacro="http://www.ros.org/wiki/xacro">
+  <!-- Tags needed for rviz to color model -->
+  <xacro:include filename="$(find pybullet_ros)/common/test/urdf/r2d2_robot/materials.urdf.xacro" />
+  <!-- hokuyo laser scanner -->
+  <xacro:include filename="$(find pybullet_ros)/common/test/urdf/laser_scanner/laser_scanner.urdf.xacro" />
+  <xacro:property name="laser_name" value="front" />
+  <xacro:hokuyo name="${laser_name}" />
   <link name="base_footprint"/>
   <link name="base_link">
@@ -24,5 +30,10 @@
     <parent link="base_footprint"/>
     <child link="base_link"/>
-    <origin xyz="0 0 0" rpy="0 0 -1.57075" />
+    <origin xyz="0 0 0.4345" rpy="0 0 -1.57075" />
+  </joint>
+  <joint name="base_link_to_laser_body" type="fixed">
+    <parent link="base_link"/>
+    <child link="${laser_name}_laser_body"/>
+    <origin xyz="0 0.25 -0.4" rpy="0 0 1.5707963" />
   </joint>
   <link name="right_leg">
@@ -224,126 +235,4 @@
     <joint_properties damping="0.0" friction="0.0"/>
   </joint>
-  <joint name="gripper_extension" type="prismatic">
-    <axis xyz="1 0 0"/>
-    <parent link="base_link"/>
-    <child link="gripper_pole"/>
-    <limit effort="1000.0" lower="-0.38" upper="0" velocity="0.5"/>
-    <origin rpy="0 0 1.57075" xyz="0 0.19 .2"/>
-  </joint>
-  <link name="gripper_pole">
-    <visual>
-      <geometry>
-        <cylinder length="0.2" radius=".01"/>
-      </geometry>
-      <origin rpy="0 1.57075 0 " xyz="0.1 0 0"/>
-      <material name="Gray">
-        <color rgba=".7 .7 .7 1"/>
-      </material>
-    </visual>
-    <collision>
-      <geometry>
-        <cylinder length="0.2" radius=".01"/>
-      </geometry>
-      <origin rpy="0 1.57075 0 " xyz="0.1 0 0"/>
-    </collision>
-    <inertial>
-      <mass value="0.05"/>
-      <inertia ixx="1.0" ixy="0.0" ixz="0.0" iyy="1.0" iyz="0.0" izz="1.0"/>
-    </inertial>
-  </link>
-  <joint name="left_gripper_joint" type="revolute">
-    <axis xyz="0 0 1"/>
-    <limit effort="1000.0" lower="0.0" upper="0.548" velocity="0.5"/>
-    <origin rpy="0 0 0" xyz="0.2 0.02 0"/>
-    <parent link="gripper_pole"/>
-    <child link="left_gripper"/>
-  </joint>
-  <link name="left_gripper">
-    <visual>
-      <origin rpy="0.0 0 0" xyz="0 0 0"/>
-      <geometry>
-        <mesh filename="l_finger.stl"/>
-      </geometry>
-    </visual>
-    <collision>
-      <geometry>
-        <mesh filename="l_finger.stl"/>
-      </geometry>
-      <origin rpy="0.0 0 0" xyz="0 0 0"/>
-    </collision>
-    <inertial>
-      <mass value="0.05"/>
-      <inertia ixx="1.0" ixy="0.0" ixz="0.0" iyy="1.0" iyz="0.0" izz="1.0"/>
-    </inertial>
-  </link>
-  <joint name="left_tip_joint" type="fixed">
-    <parent link="left_gripper"/>
-    <child link="left_tip"/>
-  </joint>
-  <link name="left_tip">
-    <visual>
-      <origin rpy="0.0 0 0" xyz="0.09137 0.00495 0"/>
-      <geometry>
-        <mesh filename="l_finger_tip.stl"/>
-      </geometry>
-    </visual>
-    <collision>
-      <geometry>
-        <mesh filename="l_finger_tip.stl"/>
-      </geometry>
-      <origin rpy="0.0 0 0" xyz="0.09137 0.00495 0"/>
-    </collision>
-    <inertial>
-      <mass value="0.05"/>
-      <inertia ixx="1.0" ixy="0.0" ixz="0.0" iyy="1.0" iyz="0.0" izz="1.0"/>
-    </inertial>
-  </link>
-  <joint name="right_gripper_joint" type="revolute">
-    <axis xyz="0 0 -1"/>
-    <limit effort="1000.0" lower="0.0" upper="0.548" velocity="0.5"/>
-    <origin rpy="0 0 0" xyz="0.2 -0.02 0"/>
-    <parent link="gripper_pole"/>
-    <child link="right_gripper"/>
-  </joint>
-  <link name="right_gripper">
-    <visual>
-      <origin rpy="-3.1415 0 0" xyz="0 0 0"/>
-      <geometry>
-        <mesh filename="l_finger.stl"/>
-      </geometry>
-    </visual>
-    <collision>
-      <geometry>
-        <mesh filename="l_finger.stl"/>
-      </geometry>
-      <origin rpy="-3.1415 0 0" xyz="0 0 0"/>
-    </collision>
-    <inertial>
-      <mass value="0.05"/>
-      <inertia ixx="1.0" ixy="0.0" ixz="0.0" iyy="1.0" iyz="0.0" izz="1.0"/>
-    </inertial>
-  </link>
-  <joint name="right_tip_joint" type="fixed">
-    <parent link="right_gripper"/>
-    <child link="right_tip"/>
-  </joint>
-  <link name="right_tip">
-    <visual>
-      <origin rpy="-3.1415 0 0" xyz="0.09137 0.00495 0"/>
-      <geometry>
-        <mesh filename="l_finger_tip.stl"/>
-      </geometry>
-    </visual>
-    <collision>
-      <geometry>
-        <mesh filename="l_finger_tip.stl"/>
-      </geometry>
-      <origin rpy="-3.1415 0 0" xyz="0.09137 0.00495 0"/>
-    </collision>
-    <inertial>
-      <mass value="0.05"/>
-      <inertia ixx="1.0" ixy="0.0" ixz="0.0" iyy="1.0" iyz="0.0" izz="1.0"/>
-    </inertial>
-  </link>
   <link name="head">
     <visual>
@@ -363,10 +252,10 @@
     </inertial>
   </link>
-  <joint name="head_swivel" type="continuous">
+  <joint name="head_swivel" type="revolute">
     <parent link="base_link"/>
     <child link="head"/>
     <axis xyz="0 0 1"/>
     <origin xyz="0 0 0.3"/>
-<limit effort="1000.0" lower="-0.38" upper="0" velocity="0.5"/>
+    <limit effort="1500.0" lower="-1.5707963" upper="1.5707963" velocity="100.0"/>
   </joint>
   <link name="box">
@@ -392,3 +281,4 @@
     <origin xyz="0 0.1214 0.1214"/>
   </joint>
+  <!-- laser scanner -->
 </robot>

Commit message: modify r2d2 urdf model to match with ROS conventions (x forward, y left)

File: common/test/urdf/r2d2_robot/r2d2.urdf.xacro (robot description, xacro)
@@ -7,5 +7,5 @@
   <xacro:property name="laser_name" value="front" />
   <xacro:hokuyo name="${laser_name}" />
-  <link name="base_footprint"/>
+  <xacro:property name="M_PI" value="3.141592653589793" />
   <link name="base_link">
     <visual>
@@ -13,7 +13,5 @@
         <cylinder length="0.6" radius="0.2"/>
       </geometry>
-      <material name="blue">
-        <color rgba="0 0 .8 1"/>
-      </material>
+      <material name="blue"/>
     </visual>
     <collision>
@@ -27,33 +25,26 @@
     </inertial>
   </link>
-  <joint name="footprint_to_base_link" type="fixed">
-    <parent link="base_footprint"/>
-    <child link="base_link"/>
-    <origin xyz="0 0 0.4345" rpy="0 0 -1.57075" />
-  </joint>
   <joint name="base_link_to_laser_body" type="fixed">
     <parent link="base_link"/>
     <child link="${laser_name}_laser_body"/>
-    <origin xyz="0 0.25 -0.4" rpy="0 0 1.5707963" />
+    <origin xyz="0.25 0.0 -0.4" rpy="0 0 0" />
   </joint>
   <link name="right_leg">
     <visual>
       <geometry>
-        <box size="0.6 .2 .1"/>
-      </geometry>
-      <origin rpy="0 1.57075 0" xyz="0 0 -0.3"/>
-      <material name="white">
-        <color rgba="1 1 1 1"/>
-      </material>
-    </visual>
-    <collision>
-      <geometry>
-        <box size="0.6 .2 .1"/>
-      </geometry>
-      <origin rpy="0 1.57075 0" xyz="0 0 -0.3"/>
-    </collision>
-    <inertial>
-      <mass value="10"/>
-      <origin rpy="0 1.57075 0" xyz="0 0 -0.3"/>
+        <box size="0.6 0.1 0.2"/>
+      </geometry>
+      <origin rpy="0 ${M_PI/2.0} 0" xyz="0 0 -0.3"/>
+      <material name="white"/>
+    </visual>
+    <collision>
+      <geometry>
+        <box size="0.6 0.1 0.2"/>
+      </geometry>
+      <origin rpy="0 ${M_PI/2.0} 0" xyz="0 0 -0.3"/>
+    </collision>
+    <inertial>
+      <mass value="10"/>
+      <origin rpy="0 ${M_PI/2.0} 0" xyz="0 0 -0.3"/>
       <inertia ixx="1.0" ixy="0.0" ixz="0.0" iyy="1.0" iyz="0.0" izz="1.0"/>
     </inertial>
@@ -62,16 +53,16 @@
     <parent link="base_link"/>
     <child link="right_leg"/>
-    <origin xyz="0.22 0 .25"/>
+    <origin xyz="0 -0.22 0.25"/>
   </joint>
   <link name="right_base">
     <visual>
       <geometry>
-        <box size=".1 0.4 .1"/>
-      </geometry>
-      <material name="white"/>
-    </visual>
-    <collision>
-      <geometry>
-        <box size=".1 0.4 .1"/>
+        <box size="0.4 0.1 0.1"/>
+      </geometry>
+      <material name="white"/>
+    </visual>
+    <collision>
+      <geometry>
+        <box size="0.4 0.1 0.1"/>
       </geometry>
     </collision>
@@ -88,15 +79,16 @@
   <link name="right_front_wheel">
     <visual>
-      <geometry>
-        <cylinder length=".1" radius="0.035"/>
-      </geometry>
-      <material name="black">
-        <color rgba="0.5 0.5 0.5 1"/>
-      </material>
-    </visual>
-    <collision>
-      <geometry>
-        <cylinder length=".1" radius="0.035"/>
-      </geometry>
+      <origin rpy="${M_PI/2.0} 0 0" xyz="0 0 0"/>
+      <geometry>
+        <cylinder length="0.1" radius="0.035"/>
+      </geometry>
+      <material name="black"/>
+    </visual>
+    <collision>
+      <origin rpy="${M_PI/2.0} 0 0" xyz="0 0 0"/>
+      <geometry>
+        <cylinder length="0.1" radius="0.035"/>
+      </geometry>
+      <material name="black"/>
     </collision>
     <inertial>
@@ -109,5 +101,5 @@
     <parent link="right_base"/>
     <child link="right_front_wheel"/>
-    <origin rpy="0 1.57075 0" xyz="0 0.133333333333 -0.085"/>
+    <origin rpy="0 0 0" xyz="0.133333333333 0 -0.085"/>
     <limit effort="100" velocity="100"/>
     <joint_properties damping="0.0" friction="0.0"/>
@@ -115,13 +107,16 @@
   <link name="right_back_wheel">
     <visual>
-      <geometry>
-        <cylinder length=".1" radius="0.035"/>
-      </geometry>
-      <material name="black"/>
-    </visual>
-    <collision>
-      <geometry>
-        <cylinder length=".1" radius="0.035"/>
-      </geometry>
+      <origin rpy="${M_PI/2.0} 0 0" xyz="0 0 0"/>
+      <geometry>
+        <cylinder length="0.1" radius="0.035"/>
+      </geometry>
+      <material name="black"/>
+    </visual>
+    <collision>
+      <origin rpy="${M_PI/2.0} 0 0" xyz="0 0 0"/>
+      <geometry>
+        <cylinder length="0.1" radius="0.035"/>
+      </geometry>
+      <material name="black"/>
     </collision>
     <inertial>
@@ -132,28 +127,28 @@
   <joint name="right_back_wheel_joint" type="continuous">
     <axis xyz="0 0 1"/>
+    <origin rpy="0 0 0" xyz="-0.133333333333 0 -0.085"/>
+    <limit effort="100" velocity="100"/>
+    <joint_properties damping="0.0" friction="0.0"/>
     <parent link="right_base"/>
     <child link="right_back_wheel"/>
-    <origin rpy="0 1.57075 0" xyz="0 -0.133333333333 -0.085"/>
-    <limit effort="100" velocity="100"/>
-    <joint_properties damping="0.0" friction="0.0"/>
   </joint>
   <link name="left_leg">
     <visual>
       <geometry>
-        <box size="0.6 .2 .1"/>
-      </geometry>
-      <origin rpy="0 1.57075 0" xyz="0 0 -0.3"/>
-      <material name="white"/>
-    </visual>
-    <collision>
-      <geometry>
-        <box size="0.6 .2 .1"/>
-      </geometry>
-      <origin rpy="0 1.57075 0" xyz="0 0 -0.3"/>
-    </collision>
-    <inertial>
-      <mass value="10"/>
-      <inertia ixx="1.0" ixy="0.0" ixz="0.0" iyy="1.0" iyz="0.0" izz="1.0"/>
-       <origin rpy="0 1.57075 0" xyz="0 0 -0.3"/>
+        <box size="0.6 0.1 0.2"/>
+      </geometry>
+      <origin rpy="0 ${M_PI/2.0} 0" xyz="0 0 -0.3"/>
+      <material name="white"/>
+    </visual>
+    <collision>
+      <geometry>
+        <box size="0.6 0.1 0.2"/>
+      </geometry>
+      <origin rpy="0 ${M_PI/2.0} 0" xyz="0 0 -0.3"/>
+    </collision>
+    <inertial>
+      <mass value="10"/>
+      <inertia ixx="1.0" ixy="0.0" ixz="0.0" iyy="1.0" iyz="0.0" izz="1.0"/>
+      <origin rpy="0 ${M_PI/2.0} 0" xyz="0 0 -0.3"/>
     </inertial>
   </link>
@@ -161,16 +156,16 @@
     <parent link="base_link"/>
     <child link="left_leg"/>
-    <origin xyz="-0.22 0 .25"/>
+    <origin xyz="0 0.22 0.25"/>
   </joint>
   <link name="left_base">
     <visual>
       <geometry>
-        <box size=".1 0.4 .1"/>
-      </geometry>
-      <material name="white"/>
-    </visual>
-    <collision>
-      <geometry>
-        <box size=".1 0.4 .1"/>
+        <box size="0.4 0.1 0.1"/>
+      </geometry>
+      <material name="white"/>
+    </visual>
+    <collision>
+      <geometry>
+        <box size="0.4 0.1 0.1"/>
       </geometry>
     </collision>
@@ -187,12 +182,14 @@
   <link name="left_front_wheel">
     <visual>
-      <geometry>
-        <cylinder length=".1" radius="0.035"/>
-      </geometry>
-      <material name="black"/>
-    </visual>
-    <collision>
-      <geometry>
-        <cylinder length=".1" radius="0.035"/>
+      <origin rpy="${M_PI/2.0} 0 0" xyz="0 0 0"/>
+      <geometry>
+        <cylinder length="0.1" radius="0.035"/>
+      </geometry>
+      <material name="black"/>
+    </visual>
+    <collision>
+      <origin rpy="${M_PI/2.0} 0 0" xyz="0 0 0"/>
+      <geometry>
+        <cylinder length="0.1" radius="0.035"/>
       </geometry>
     </collision>
@@ -206,5 +203,5 @@
     <parent link="left_base"/>
     <child link="left_front_wheel"/>
-    <origin rpy="0 1.57075 0" xyz="0 0.133333333333 -0.085"/>
+    <origin rpy="0 0 0" xyz="0.133333333333 0 -0.085"/>
     <limit effort="100" velocity="100"/>
     <joint_properties damping="0.0" friction="0.0"/>
@@ -212,12 +209,14 @@
   <link name="left_back_wheel">
     <visual>
-      <geometry>
-        <cylinder length=".1" radius="0.035"/>
-      </geometry>
-      <material name="black"/>
-    </visual>
-    <collision>
-      <geometry>
-        <cylinder length=".1" radius="0.035"/>
+      <origin rpy="${M_PI/2.0} 0 0" xyz="0 0 0"/>
+      <geometry>
+        <cylinder length="0.1" radius="0.035"/>
+      </geometry>
+      <material name="black"/>
+    </visual>
+    <collision>
+      <origin rpy="${M_PI/2.0} 0 0" xyz="0 0 0"/>
+      <geometry>
+        <cylinder length="0.1" radius="0.035"/>
       </geometry>
     </collision>
@@ -231,5 +230,5 @@
     <parent link="left_base"/>
     <child link="left_back_wheel"/>
-    <origin rpy="0 1.57075 0" xyz="0 -0.133333333333 -0.085"/>
+    <origin rpy="0 0 0" xyz="-0.133333333333 0 -0.085"/>
     <limit effort="100" velocity="100"/>
     <joint_properties damping="0.0" friction="0.0"/>
@@ -257,5 +256,5 @@
     <axis xyz="0 0 1"/>
     <origin xyz="0 0 0.3"/>
-    <limit effort="1500.0" lower="-1.5707963" upper="1.5707963" velocity="100.0"/>
+    <limit effort="1500.0" lower="-${M_PI/2.0}" upper="${M_PI/2.0}" velocity="100.0"/>
   </joint>
   <link name="box">
@@ -279,6 +278,5 @@
     <parent link="head"/>
     <child link="box"/>
-    <origin xyz="0 0.1214 0.1214"/>
-  </joint>
-  <!-- laser scanner -->
+    <origin xyz="0.1214 0 0.1214"/>
+  </joint>
 </robot>
