Commit message: Added a new bottom heavy R2D2 to stop from toppling

File: common/test/urdf/r2d2_robot/r2d2_bottom_heavy.urdf (robot description, URDF)
Before this commit: robot r2d2, 11 links, 11 joints
Links:
- added link front_laser; collision cylinder length=0.029 radius=0.021; visual cylinder length=0.029 radius=0.021
- added link front_laser_body; collision box size=0.05 0.05 0.041; visual box size=0.05 0.05 0.041
- link base_link: mass 10 -> 5
- link head: mass 10 -> 5
- link left_back_wheel: mass 1 -> 5
- link left_base: mass 10 -> 20
- link left_front_wheel: mass 1 -> 5
- link left_leg: mass 10 -> 5
- link right_back_wheel: mass 1 -> 5
- link right_base: mass 10 -> 20
- link right_front_wheel: mass 1 -> 5
- link right_leg: mass 10 -> 5
Joints:
- added joint front_laser_body_to_front_laser: type fixed, parent front_laser_body, child front_laser, origin xyz=0 0 0.0615 rpy=0 0 0
- joint base_link_to_laser_body: child ${laser_name}_laser_body -> front_laser_body
- joint head_swivel: limit lower=-${M_PI/2.0} upper=${M_PI/2.0} effort=1500.0 velocity=100.0 -> lower=-1.5707963267948966 upper=1.5707963267948966 effort=1500.0 velocity=100.0

File: common/test/urdf/r2d2_robot/r2d2_bottom_heavy.urdf.xacro (robot description, xacro)
@@ -23,5 +23,5 @@
     </collision>
     <inertial>
-      <mass value="10"/>
+      <mass value="5"/>
       <inertia ixx="1.0" ixy="0.0" ixz="0.0" iyy="1.0" iyz="0.0" izz="1.0"/>
     </inertial>
@@ -47,5 +47,5 @@
     </collision>
     <inertial>
-      <mass value="10"/>
+      <mass value="5"/>
       <origin rpy="0 ${M_PI/2.0} 0" xyz="0 0 -0.3"/>
       <inertia ixx="1.0" ixy="0.0" ixz="0.0" iyy="1.0" iyz="0.0" izz="1.0"/>
@@ -70,5 +70,5 @@
     </collision>
     <inertial>
-      <mass value="10"/>
+      <mass value="20"/>
       <inertia ixx="1.0" ixy="0.0" ixz="0.0" iyy="1.0" iyz="0.0" izz="1.0"/>
     </inertial>
@@ -95,5 +95,5 @@
     </collision>
     <inertial>
-      <mass value="1"/>
+      <mass value="5"/>
       <inertia ixx="1.0" ixy="0.0" ixz="0.0" iyy="1.0" iyz="0.0" izz="1.0"/>
     </inertial>
@@ -123,5 +123,5 @@
     </collision>
     <inertial>
-      <mass value="1"/>
+      <mass value="5"/>
       <inertia ixx="1.0" ixy="0.0" ixz="0.0" iyy="1.0" iyz="0.0" izz="1.0"/>
     </inertial>
@@ -150,5 +150,5 @@
     </collision>
     <inertial>
-      <mass value="10"/>
+      <mass value="5"/>
       <inertia ixx="1.0" ixy="0.0" ixz="0.0" iyy="1.0" iyz="0.0" izz="1.0"/>
       <origin rpy="0 ${M_PI/2.0} 0" xyz="0 0 -0.3"/>
@@ -173,5 +173,5 @@
     </collision>
     <inertial>
-      <mass value="10"/>
+      <mass value="20"/>
       <inertia ixx="1.0" ixy="0.0" ixz="0.0" iyy="1.0" iyz="0.0" izz="1.0"/>
     </inertial>
@@ -197,5 +197,5 @@
     </collision>
     <inertial>
-      <mass value="1"/>
+      <mass value="5"/>
       <inertia ixx="1.0" ixy="0.0" ixz="0.0" iyy="1.0" iyz="0.0" izz="1.0"/>
     </inertial>
@@ -224,5 +224,5 @@
     </collision>
     <inertial>
-      <mass value="1"/>
+      <mass value="5"/>
       <inertia ixx="1.0" ixy="0.0" ixz="0.0" iyy="1.0" iyz="0.0" izz="1.0"/>
     </inertial>
@@ -249,5 +249,5 @@
     </collision>
     <inertial>
-      <mass value="10"/>
+      <mass value="5"/>
       <inertia ixx="1.0" ixy="0.0" ixz="0.0" iyy="1.0" iyz="0.0" izz="1.0"/>
     </inertial>

File: common/test/urdf/r2d2_robot/r2d2_small.urdf (robot description, URDF)
Before this commit: robot r2d2, 11 links, 11 joints
Links:
- added link front_laser; collision cylinder length=0.029 radius=0.021; visual cylinder length=0.029 radius=0.021
- added link front_laser_body; collision box size=0.05 0.05 0.041; visual box size=0.05 0.05 0.041
- link base_link: mass 10 -> 5
- link head: mass 10 -> 5
- link left_back_wheel: mass 1 -> 5
- link left_base: mass 10 -> 20
- link left_front_wheel: mass 1 -> 5
- link left_leg: mass 10 -> 5
- link right_back_wheel: mass 1 -> 5
- link right_base: mass 10 -> 20
- link right_front_wheel: mass 1 -> 5
- link right_leg: mass 10 -> 5
Joints:
- added joint front_laser_body_to_front_laser: type fixed, parent front_laser_body, child front_laser, origin xyz=0 0 0.0615 rpy=0 0 0
- joint base_link_to_laser_body: child ${laser_name}_laser_body -> front_laser_body
- joint head_swivel: limit lower=-${M_PI/2.0} upper=${M_PI/2.0} effort=1500.0 velocity=100.0 -> lower=-1.5707963267948966 upper=1.5707963267948966 effort=1500.0 velocity=100.0
